File: pcb/monolithic_200mm_288/monolithic_200mm_288.kicad_pcb (KiCad board)
At the start: 2 copper layers, 200 x 200 mm, 600 parts

Commit message: feat: monolithic 200mm single-sided SMT with 2.54mm through-hole solder pins and strain relief
Parts:
- removed the ? at (32.5, 189.0)
- removed the ? at (35.0, 189.0)
- removed the ? at (37.5, 189.0)
- removed the ? at (162.5, 189.0)
- removed the ? at (165.0, 189.0)
- removed the ? at (167.5, 189.0)
- removed the J_IN at (35.0, 194.0)
- removed the J_OUT at (165.0, 194.0)
- added ?: , MountingHole:MountingHole_2.2mm, F.Cu at (26.0, 188.5)
- added ?: , MountingHole:MountingHole_2.2mm, F.Cu at (34.0, 188.5)
- added ?: , MountingHole:MountingHole_2.2mm, F.Cu at (166.0, 188.5)
- added ?: , MountingHole:MountingHole_2.2mm, F.Cu at (174.0, 188.5)
- added J_IN: , Connector_PinHeader_2.54mm:PinHeader_1x03_P2.54mm_Vertical, F.Cu at (30.0, 194.0)
- added J_OUT: , Connector_PinHeader_2.54mm:PinHeader_1x03_P2.54mm_Vertical, F.Cu at (170.0, 194.0)
Routing:
- net DATA_289: track 154.0 -> 169.3 mm, vias 1 -> 0
- net DATA_1: track 186.3 -> 185.8 mm, vias 1 -> 0
Changed lines of the file:
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@@
     (tracks 0)
     (zones 0)
-    (modules 594)
+    (modules 592)
     (nets 292)
   )
@@
     (pad 1 thru_hole circle (at 0 0) (size 3.5 3.5) (drill 2.0) (layers *.Cu *.Mask))
   )
-  (module "Connector_JST:JST_PH_S3B-PH-SM4-TB_1x03-1MP_P2.00mm_Horizontal" (layer B.Cu)
-    (at 35.0 194.0)
-    (descr "JST PH 3-pin IN connector on Bottom")
-    (path "/J_IN")
-    (fp_text reference "J_IN" (at 0 -3.6) (layer B.SilkS)
+  (module "Connector_PinHeader_2.54mm:PinHeader_1x03_P2.54mm_Vertical" (layer F.Cu)
+    (at 30.0 194.0)
+    (descr "2.54mm Pin Header for DATA IN")
+    (path "/HDR_IN")
+    (fp_text reference "J_IN" (at 0 -3.0) (layer F.SilkS)
       (effects (font (size 0.7 0.7) (thickness 0.12)))
     )
-    (fp_text user "[IN]" (at 0 3.6) (layer B.SilkS)
+    (fp_text user "[IN]" (at 0 3.0) (layer F.SilkS)
       (effects (font (size 0.65 0.65) (thickness 0.12)))
     )
-    (pad 1 smd rect (at -2.0 0.0) (size 1.0 1.6) (layers B.Cu B.Paste B.Mask) (net 1))
-    (pad 2 smd rect (at 0.0 0.0) (size 1.0 1.6) (layers B.Cu B.Paste B.Mask) (net 3))
-    (pad 3 smd rect (at 2.0 0.0) (size 1.0 1.6) (layers B.Cu B.Paste B.Mask) (net 2))
-    (pad MP smd rect (at -3.4 -1.5) (size 1.5 1.8) (layers B.Cu B.Paste B.Mask) (net 2))
-    (pad MP smd rect (at 3.4 -1.5) (size 1.5 1.8) (layers B.Cu B.Paste B.Mask) (net 2))
-  )
-  (module "TestPoint:TestPoint_Pad_D1.5mm" (layer B.Cu)
-    (at 32.46 189.0)
-    (descr "Direct solder eyelet 5V")
-    (path "/J_IN_5V")
-    (pad 1 thru_hole circle (at 0 0) (size 2.0 2.0) (drill 1.2) (layers *.Cu *.Mask) (net 1))
-  )
-  (module "TestPoint:TestPoint_Pad_D1.5mm" (layer B.Cu)
-    (at 35.0 189.0)
-    (descr "Direct solder eyelet DAT")
-    (path "/J_IN_DAT")
-    (pad 1 thru_hole circle (at 0 0) (size 2.0 2.0) (drill 1.2) (layers *.Cu *.Mask) (net 3))
-  )
-  (module "TestPoint:TestPoint_Pad_D1.5mm" (layer B.Cu)
-    (at 37.54 189.0)
-    (descr "Direct solder eyelet GND")
-    (path "/J_IN_GND")
-    (pad 1 thru_hole circle (at 0 0) (size 2.0 2.0) (drill 1.2) (layers *.Cu *.Mask) (net 2))
-  )
-  (module "Connector_JST:JST_PH_S3B-PH-SM4-TB_1x03-1MP_P2.00mm_Horizontal" (layer B.Cu)
-    (at 165.0 194.0)
-    (descr "JST PH 3-pin OUT connector on Bottom")
-    (path "/J_OUT")
-    (fp_text reference "J_OUT" (at 0 -3.6) (layer B.SilkS)
+    (fp_text user "[IN]" (at 0 3.0) (layer B.SilkS)
+      (effects (font (size 0.65 0.65) (thickness 0.12)))
+    )
+    (fp_line (start -4.0 -1.6) (end 4.0 -1.6) (layer F.SilkS) (width 0.15))
+    (fp_line (start 4.0 -1.6) (end 4.0 1.6) (layer F.SilkS) (width 0.15))
+    (fp_line (start 4.0 1.6) (end -4.0 1.6) (layer F.SilkS) (width 0.15))
+    (fp_line (start -4.0 1.6) (end -4.0 -1.6) (layer F.SilkS) (width 0.15))
+    (fp_line (start -4.0 -1.6) (end 4.0 -1.6) (layer B.SilkS) (width 0.15))
+    (fp_line (start 4.0 -1.6) (end 4.0 1.6) (layer B.SilkS) (width 0.15))
+    (fp_line (start 4.0 1.6) (end -4.0 1.6) (layer B.SilkS) (width 0.15))
+    (fp_line (start -4.0 1.6) (end -4.0 -1.6) (layer B.SilkS) (width 0.15))
+    (pad 1 thru_hole circle (at -2.54 0) (size 2.2 2.2) (drill 1.2) (layers *.Cu *.Mask) (net 1))
+    (fp_text user "+5V" (at -2.54 -2.0) (layer F.SilkS) (effects (font (size 0.55 0.55) (thickness 0.1))))
+    (fp_text user "+5V" (at -2.54 -2.0) (layer B.SilkS) (effects (font (size 0.55 0.55) (thickness 0.1))))
+    (pad 2 thru_hole circle (at 0.0 0) (size 2.2 2.2) (drill 1.2) (layers *.Cu *.Mask) (net 3))
+    (fp_text user "DAT" (at 0.0 -2.0) (layer F.SilkS) (effects (font (size 0.55 0.55) (thickness 0.1))))
+    (fp_text user "DAT" (at 0.0 -2.0) (layer B.SilkS) (effects (font (size 0.55 0.55) (thickness 0.1))))
+    (pad 3 thru_hole circle (at 2.54 0) (size 2.2 2.2) (drill 1.2) (layers *.Cu *.Mask) (net 2))
+    (fp_text user "GND" (at 2.54 -2.0) (layer F.SilkS) (effects (font (size 0.55 0.55) (thickness 0.1))))
+    (fp_text user "GND" (at 2.54 -2.0) (layer B.SilkS) (effects (font (size 0.55 0.55) (thickness 0.1))))
+  )
+  (module "MountingHole:MountingHole_2.2mm" (layer F.Cu)
+    (at 26.0 188.5)
+    (descr "Wire Strain Relief Hole 2.2mm")
+    (path "/STRAIN_IN_1")
+    (pad 1 np_thru_hole circle (at 0 0) (size 2.2 2.2) (drill 2.2) (layers *.Mask))
+  )
+  (module "MountingHole:MountingHole_2.2mm" (layer F.Cu)
+    (at 34.0 188.5)
+    (descr "Wire Strain Relief Hole 2.2mm")
+    (path "/STRAIN_IN_2")
+    (pad 1 np_thru_hole circle (at 0 0) (size 2.2 2.2) (drill 2.2) (layers *.Mask))
+  )
+  (module "Connector_PinHeader_2.54mm:PinHeader_1x03_P2.54mm_Vertical" (layer F.Cu)
+    (at 170.0 194.0)
+    (descr "2.54mm Pin Header for DATA OUT")
+    (path "/HDR_OUT")
+    (fp_text reference "J_OUT" (at 0 -3.0) (layer F.SilkS)
       (effects (font (size 0.7 0.7) (thickness 0.12)))
     )
-    (fp_text user "[OUT]" (at 0 3.6) (layer B.SilkS)
+    (fp_text user "[OUT]" (at 0 3.0) (layer F.SilkS)
+      (effects (font (size 0.65 0.65) (thickness 0.12)))
+    )
+    (fp_text user "[OUT]" (at 0 3.0) (layer B.SilkS)
       (effects (font (size 0.65 0.65) (thickness 0.12)))
     )
-    (pad 1 smd rect (at -2.0 0.0) (size 1.0 1.6) (layers B.Cu B.Paste B.Mask) (net 1))
-    (pad 2 smd rect (at 0.0 0.0) (size 1.0 1.6) (layers B.Cu B.Paste B.Mask) (net 291))
-    (pad 3 smd rect (at 2.0 0.0) (size 1.0 1.6) (layers B.Cu B.Paste B.Mask) (net 2))
-    (pad MP smd rect (at -3.4 -1.5) (size 1.5 1.8) (layers B.Cu B.Paste B.Mask) (net 2))
-    (pad MP smd rect (at 3.4 -1.5) (size 1.5 1.8) (layers B.Cu B.Paste B.Mask) (net 2))
-  )
-  (module "TestPoint:TestPoint_Pad_D1.5mm" (layer B.Cu)
-    (at 162.46 189.0)
-    (descr "Direct solder eyelet 5V")
-    (path "/J_OUT_5V")
-    (pad 1 thru_hole circle (at 0 0) (size 2.0 2.0) (drill 1.2) (layers *.Cu *.Mask) (net 1))
-  )
-  (module "TestPoint:TestPoint_Pad_D1.5mm" (layer B.Cu)
-    (at 165.0 189.0)
-    (descr "Direct solder eyelet DAT")
-    (path "/J_OUT_DAT")
-    (pad 1 thru_hole circle (at 0 0) (size 2.0 2.0) (drill 1.2) (layers *.Cu *.Mask) (net 291))
-  )
-  (module "TestPoint:TestPoint_Pad_D1.5mm" (layer B.Cu)
-    (at 167.54 189.0)
-    (descr "Direct solder eyelet GND")
-    (path "/J_OUT_GND")
-    (pad 1 thru_hole circle (at 0 0) (size 2.0 2.0) (drill 1.2) (layers *.Cu *.Mask) (net 2))
+    (fp_line (start -4.0 -1.6) (end 4.0 -1.6) (layer F.SilkS) (width 0.15))
+    (fp_line (start 4.0 -1.6) (end 4.0 1.6) (layer F.SilkS) (width 0.15))
+    (fp_line (start 4.0 1.6) (end -4.0 1.6) (layer F.SilkS) (width 0.15))
+    (fp_line (start -4.0 1.6) (end -4.0 -1.6) (layer F.SilkS) (width 0.15))
+    (fp_line (start -4.0 -1.6) (end 4.0 -1.6) (layer B.SilkS) (width 0.15))
+    (fp_line (start 4.0 -1.6) (end 4.0 1.6) (layer B.SilkS) (width 0.15))
+    (fp_line (start 4.0 1.6) (end -4.0 1.6) (layer B.SilkS) (width 0.15))
+    (fp_line (start -4.0 1.6) (end -4.0 -1.6) (layer B.SilkS) (width 0.15))
+    (pad 1 thru_hole circle (at -2.54 0) (size 2.2 2.2) (drill 1.2) (layers *.Cu *.Mask) (net 1))
+    (fp_text user "+5V" (at -2.54 -2.0) (layer F.SilkS) (effects (font (size 0.55 0.55) (thickness 0.1))))
+    (fp_text user "+5V" (at -2.54 -2.0) (layer B.SilkS) (effects (font (size 0.55 0.55) (thickness 0.1))))
+    (pad 2 thru_hole circle (at 0.0 0) (size 2.2 2.2) (drill 1.2) (layers *.Cu *.Mask) (net 291))
+    (fp_text user "DAT" (at 0.0 -2.0) (layer F.SilkS) (effects (font (size 0.55 0.55) (thickness 0.1))))
+    (fp_text user "DAT" (at 0.0 -2.0) (layer B.SilkS) (effects (font (size 0.55 0.55) (thickness 0.1))))
+    (pad 3 thru_hole circle (at 2.54 0) (size 2.2 2.2) (drill 1.2) (layers *.Cu *.Mask) (net 2))
+    (fp_text user "GND" (at 2.54 -2.0) (layer F.SilkS) (effects (font (size 0.55 0.55) (thickness 0.1))))
+    (fp_text user "GND" (at 2.54 -2.0) (layer B.SilkS) (effects (font (size 0.55 0.55) (thickness 0.1))))
+  )
+  (module "MountingHole:MountingHole_2.2mm" (layer F.Cu)
+    (at 166.0 188.5)
+    (descr "Wire Strain Relief Hole 2.2mm")
+    (path "/STRAIN_OUT_1")
+    (pad 1 np_thru_hole circle (at 0 0) (size 2.2 2.2) (drill 2.2) (layers *.Mask))
+  )
+  (module "MountingHole:MountingHole_2.2mm" (layer F.Cu)
+    (at 174.0 188.5)
+    (descr "Wire Strain Relief Hole 2.2mm")
+    (path "/STRAIN_OUT_2")
+    (pad 1 np_thru_hole circle (at 0 0) (size 2.2 2.2) (drill 2.2) (layers *.Mask))
   )
   (module "LED_SMD:LED_WS2812B-2020_PLCC4_2.0x2.0mm" (layer F.Cu)
@@
   (segment (start 26.65 190.75) (end 16.75 189.45) (width 0.22) (layer F.Cu) (net 290))
   (segment (start 29.3 189.62) (end 17.7 189.62) (width 0.6) (layer F.Cu) (net 1))
-  (via (at 35.0 190.0) (size 0.8) (drill 0.4) (layers F.Cu B.Cu) (net 3))
-  (segment (start 35.0 194.0) (end 35.0 190.0) (width 0.3) (layer B.Cu) (net 3))
-  (segment (start 35.0 190.0) (end 10.95 9.25) (width 0.22) (layer F.Cu) (net 3))
-  (via (at 165.0 190.0) (size 0.8) (drill 0.4) (layers F.Cu B.Cu) (net 291))
-  (segment (start 15.05 190.75) (end 165.0 190.0) (width 0.22) (layer F.Cu) (net 291))
-  (segment (start 165.0 190.0) (end 165.0 194.0) (width 0.3) (layer B.Cu) (net 291))
+  (segment (start 30.0 194.0) (end 30.0 180.0) (width 0.3) (layer F.Cu) (net 3))
+  (segment (start 30.0 180.0) (end 10.95 9.25) (width 0.22) (layer F.Cu) (net 3))
+  (segment (start 15.05 190.75) (end 170.0 180.0) (width 0.22) (layer F.Cu) (net 291))
+  (segment (start 170.0 180.0) (end 170.0 194.0) (width 0.3) (layer F.Cu) (net 291))
   (zone (net 2) (net_name "GND") (layer B.Cu) (hatch edge 0.5)
     (connect_pads yes (clearance 0.25))
